Commit message: FIxed IGN model for simulation

File: models/imu_brick_v2/imu_brick_v2.xacro (robot description, xacro)
@@ -17,5 +17,5 @@
             <visual>
                 <geometry>
-                    <mesh filename="package://idmind_imu/model/imu_brick_v2/imu_brick_v2.stl" scale="0.001 0.001 0.001"/>
+                    <mesh filename="/home/cneves/ros2_youship/src/idmind_imu/models/imu_brick_v2/imu_brick_v2.stl" scale="0.001 0.001 0.001"/>
                 </geometry>
                 <material name="black" />
@@ -46,13 +46,6 @@
                 <update_rate>25</update_rate>
                 <visualize>false</visualize>
-                <topic>__default_topic__</topic>
-                <plugin filename="libgazebo_ros_imu_sensor.so" name="imu_plugin">
-                    <topicName>idmind_imu/imu</topicName>
-                    <bodyName>imu</bodyName>
-                    <updateRateHZ>20.0</updateRateHZ>
-                    <gaussianNoise>0.001</gaussianNoise>
-                    <xyzOffset>0 0 0</xyzOffset>
-                    <rpyOffset>0 0 0</rpyOffset>
-                    <frameName>${prefix}imu</frameName>
+                <topic>imu</topic>
+                <plugin filename="libignition-gazebo-imu-system.so" name="ignition::gazebo::systems::Imu">
                 </plugin>
                 <pose>0 0 0 0 0 0</pose>

Commit message: Fixed model to work for ROS2 simulations

File: models/imu_brick_v2/imu_brick_v2.xacro (robot description, xacro)
@@ -17,5 +17,5 @@
             <visual>
                 <geometry>
-                    <mesh filename="/home/cneves/ros2_youship/src/idmind_imu/models/imu_brick_v2/imu_brick_v2.stl" scale="0.001 0.001 0.001"/>
+                    <mesh filename="file:///home/cneves/ros2_youship/src/idmind_imu/models/imu_brick_v2/imu_brick_v2.dae" /> <!--scale="0.001 0.001 0.001"/-->
                 </geometry>
                 <material name="black" />

Commit message: Improvements to the model

File: models/imu_brick_v2/imu_brick_v2.xacro (robot description, xacro)
@@ -14,5 +14,5 @@
         <xacro:property name="imu_length" value="0.031" />
         <xacro:property name="imu_mass" value="0.010" />
-        <link name="${imu_name}">
+        <link name="${prefix}_${imu_name}">
             <visual>
                 <geometry>
@@ -36,15 +36,15 @@
         <joint name="base_to_${imu_name}" type="fixed">
             <parent link="${parent}"/>
-            <child link="${imu_name}"/>
+            <child link="${prefix}_${imu_name}"/>
             <xacro:insert_block name="xyz" />
         </joint>
-        <gazebo reference="${imu_name}">
+        <gazebo reference="${prefix}_${imu_name}">
             <material>Gazebo/Black</material>
             <gravity>true</gravity>
-            <sensor name="imu_sensor" type="imu">
+            <sensor name="${prefix}_imu_sensor" type="imu">
                 <always_on>true</always_on>
                 <update_rate>25</update_rate>
                 <visualize>false</visualize>
-                <topic>imu</topic>
+                <topic>${prefix}imu</topic>
                 <plugin filename="libignition-gazebo-imu-system.so" name="ignition::gazebo::systems::Imu">
                 </plugin>

Commit message: Added parameters to Gazebo model

File: models/imu_brick_v2/imu_brick_v2.xacro (robot description, xacro)
@@ -14,5 +14,5 @@
         <xacro:property name="imu_length" value="0.031" />
         <xacro:property name="imu_mass" value="0.010" />
-        <link name="${prefix}_${imu_name}">
+        <link name="${prefix}/${imu_name}">
             <visual>
                 <geometry>
@@ -36,8 +36,8 @@
         <joint name="base_to_${imu_name}" type="fixed">
             <parent link="${parent}"/>
-            <child link="${prefix}_${imu_name}"/>
+            <child link="${prefix}/${imu_name}"/>
             <xacro:insert_block name="xyz" />
         </joint>
-        <gazebo reference="${prefix}_${imu_name}">
+        <gazebo reference="${prefix}/${imu_name}">
             <material>Gazebo/Black</material>
             <gravity>true</gravity>
@@ -47,6 +47,7 @@
                 <visualize>false</visualize>
                 <topic>${prefix}/imu</topic>
+                <gz_frame_id>${prefix}/imu</gz_frame_id>
+                <ignition_frame_id>${prefix}/imu</ignition_frame_id>
                 <plugin filename="libignition-gazebo-imu-system.so" name="ignition::gazebo::systems::Imu">
-                    <frame_name>imu</frame_name>
                 </plugin>
                 <pose>0 0 0 0 0 0</pose>

Commit message: Minor adjustment to lidar model

File: models/imu_brick_v2/imu_brick_v2.xacro (robot description, xacro)
@@ -14,5 +14,5 @@
         <xacro:property name="imu_length" value="0.031" />
         <xacro:property name="imu_mass" value="0.010" />
-        <link name="${prefix}/${imu_name}">
+        <link name="${prefix}${imu_name}">
             <visual>
                 <geometry>
@@ -34,10 +34,10 @@
             </inertial>
         </link>
-        <joint name="base_to_${imu_name}" type="fixed">
-            <parent link="${parent}"/>
-            <child link="${prefix}/${imu_name}"/>
+        <joint name="${prefix}${parent}_to_${imu_name}" type="fixed">
+            <parent link="${prefix}${parent}"/>
+            <child link="${prefix}${imu_name}"/>
             <xacro:insert_block name="xyz" />
         </joint>
-        <gazebo reference="${prefix}/${imu_name}">
+        <gazebo reference="${prefix}${imu_name}">
             <material>Gazebo/Black</material>
             <gravity>true</gravity>
@@ -46,7 +46,7 @@
                 <update_rate>25</update_rate>
                 <visualize>false</visualize>
-                <topic>${prefix}/imu</topic>
-                <gz_frame_id>${prefix}/imu</gz_frame_id>
-                <ignition_frame_id>${prefix}/imu</ignition_frame_id>
+                <topic>${prefix}imu</topic>
+                <gz_frame_id>${prefix}imu</gz_frame_id>
+                <ignition_frame_id>${prefix}imu</ignition_frame_id>
                 <imu>
                 <angular_velocity>

Commit message: Minor mesh change

File: models/imu_brick_v2/imu_brick_v2.xacro (robot description, xacro)
@@ -17,5 +17,5 @@
             <visual>
                 <geometry>
-                    <mesh filename="file:///home/cneves/ros2_youship/src/idmind_imu/models/imu_brick_v2/imu_brick_v2.dae" /> <!--scale="0.001 0.001 0.001"/-->
+                    <mesh filename="package://idmind_imu/models/imu_brick_v2/imu_brick_v2.dae" /> <!--scale="0.001 0.001 0.001"/-->
                 </geometry>
                 <material name="black" />

Commit message: Minor changes to imu_brick model and mesh

File: models/imu_brick_v2/imu_brick_v2.xacro (robot description, xacro)
@@ -9,5 +9,5 @@
     </xacro:macro>
     <!-- TINKERFORGE IMU BRICK V2 -->
-    <xacro:macro name="imu_brick_v2" params="imu_name parent prefix *xyz">
+    <xacro:macro name="imu_brick_v2" params="imu_name parent prefix imu_topic:='imu_node/imu' *xyz">
         <xacro:property name="imu_height" value="0.01" />
         <xacro:property name="imu_width" value="0.031" />
@@ -17,5 +17,6 @@
             <visual>
                 <geometry>
-                    <mesh filename="package://idmind_imu/models/imu_brick_v2/imu_brick_v2.dae" /> <!--scale="0.001 0.001 0.001"/-->
+                    <!-- <mesh filename="package://idmind_imu/models/imu_brick_v2/imu_brick_v2.stl" scale="1 1 1"/> -->
+                    <mesh filename="/home/cneves/ros2_harmony/src/idmind_imu/models/imu_brick_v2/imu_brick_v2.stl" scale="1 1 1"/>
                 </geometry>
                 <material name="black" />
@@ -42,11 +43,11 @@
             <material>Gazebo/Black</material>
             <gravity>true</gravity>
-            <sensor name="${prefix}_imu_sensor" type="imu">
+            <sensor name="${prefix}imu_sensor" type="imu">
                 <always_on>true</always_on>
                 <update_rate>25</update_rate>
                 <visualize>false</visualize>
-                <topic>${prefix}imu</topic>
+                <topic>${prefix}${imu_topic}</topic>
                 <gz_frame_id>${prefix}imu</gz_frame_id>
-                <ignition_frame_id>${prefix}imu</ignition_frame_id>
+                <!-- <ignition_frame_id>${prefix}imu</ignition_frame_id> -->
                 <imu>
                 <angular_velocity>

Commit message: Minor updates to model

File: models/imu_brick_v2/imu_brick_v2.xacro (robot description, xacro)
@@ -18,7 +18,7 @@
                 <geometry>
                     <!-- <mesh filename="package://idmind_imu/models/imu_brick_v2/imu_brick_v2.stl" scale="1 1 1"/> -->
-                    <mesh filename="/home/cneves/ros2_harmony/src/idmind_imu/models/imu_brick_v2/imu_brick_v2.stl" scale="1 1 1"/>
+                    <mesh filename="/home/cneves/ros2_harmony/src/idmind_imu/models/imu_brick_v2/imu_brick_v2.stl"  scale="1 1 1" />
                 </geometry>
-                <material name="black" />
+                <material name="red" />
 	            <origin rpy="0 0 0" xyz="0 0 0"/>
             </visual>

Commit message: Updated ImUBrick model mesh

File: models/imu_brick_v2/imu_brick_v2.xacro (robot description, xacro)
@@ -17,6 +17,5 @@
             <visual>
                 <geometry>
-                    <!-- <mesh filename="package://idmind_imu/models/imu_brick_v2/imu_brick_v2.stl" scale="1 1 1"/> -->
-                    <mesh filename="/home/cneves/ros2_harmony/src/idmind_imu/models/imu_brick_v2/imu_brick_v2.stl"  scale="1 1 1" />
+                    <mesh filename="package://idmind_imu/models/imu_brick_v2/imu_brick_v2.stl"  scale="1 1 1" />
                 </geometry>
                 <material name="red" />
